Commit message: feat(osr_simplified): simplify model by removing camara and tunning laser to match RPLIDAR A2M& specs

File: osr_gazebo/urdf/osr_simplified.urdf.xacro (robot description, xacro)
@@ -450,5 +450,5 @@
                 <cylinder radius="0.03" length="0.04"/>
             </geometry>
-            <material name="red"/>
+            <material name="blue"/>
         </visual>
         <collision>
@@ -466,6 +466,6 @@
                 <scan>
                     <horizontal>
-                        <samples>360</samples>
-                        <resolution>2</resolution>
+                        <samples>720</samples>
+                        <resolution>1</resolution> <!--(max_angle-min_angle)/samples * resolution -->
                         <min_angle>-3.14159</min_angle>
                         <max_angle>3.14159</max_angle>
@@ -474,12 +474,14 @@
                 <range>
                     <min>0.3</min>
-                    <max>12</max>
+                    <max>12.0</max>
                     <resolution>0.01</resolution>
                 </range>
+                <noise>
+                    <type>gaussian</type>
+                    <mean>0.0</mean>
+                    <stddev>0.01</stddev>
+                </noise>
             </ray>
             <plugin name="laser_controller" filename="libgazebo_ros_ray_sensor.so">
-                <ros>
-                    <argument>~/out:=scan</argument>
-                </ros>
                 <output_type>sensor_msgs/LaserScan</output_type>
                 <frame_name>laser_frame</frame_name>
@@ -487,45 +489,3 @@
         </sensor>
     </gazebo>
-    <joint name="camera_joint" type="fixed">
-        <parent link="base_link"/>
-        <child link="camera_link"/>
-        <origin xyz="0.305 0 0.08" rpy="0 0 0"/>
-    </joint>
-    <link name="camera_link">
-        <visual>
-            <geometry>
-                <box size="0.010 0.03 0.03"/>
-            </geometry>
-            <material name="red"/>
-        </visual>
-    </link>
-    <joint name="camera_optical_joint" type="fixed">
-        <parent link="camera_link"/>
-        <child link="camera_link_optical"/>
-        <origin xyz="0 0 0" rpy="${-pi/2} 0 ${-pi/2}"/>
-    </joint>
-    <link name="camera_link_optical"></link>
-    <gazebo reference="camera_link">
-        <material>Gazebo/Red</material>
-        <sensor name="camera" type="camera">
-            <pose> 0 0 0 0 0 0 </pose>
-            <visualize>false</visualize>
-            <update_rate>10</update_rate>
-            <camera>
-                <horizontal_fov>1.089</horizontal_fov>
-                <image>
-                    <format>R8G8B8</format>
-                    <width>640</width>
-                    <height>480</height>
-                </image>
-                <clip>
-                    <near>0.05</near>
-                    <far>8.0</far>
-                </clip>
-            </camera>
-            <plugin name="camera_controller" filename="libgazebo_ros_camera.so">
-                <frame_name>camera_link_optical</frame_name>
-            </plugin>
-        </sensor>
-    </gazebo>
 </robot>

Commit message: Prepare urdf script for session2

File: osr_gazebo/urdf/osr_simplified.urdf.xacro (robot description, xacro)
@@ -1,9 +1,9 @@
 <?xml version="1.0" ?>
 <robot xmlns:xacro="http://www.ros.org/wiki/xacro" name="rover">
+    <xacro:include filename="$(find osr_gazebo)/urdf/gazebo.urdf.xacro"/>
+    <xacro:include filename="$(find osr_gazebo)/urdf/insert_transmission.urdf.xacro"/>
+    <!-- Add colors here -->
     <material name="black">
         <color rgba="0.1 0.1 0.1 1.0"/>
-    </material>
-    <material name="blue">
-        <color rgba="0 0 1 0.5"/>
     </material>
     <material name="sky_blue">
@@ -16,6 +16,5 @@
       <color rgba="0.5451 0.2706 0.0745 1"/>
     </material>
-    <xacro:include filename="$(find osr_gazebo)/urdf/gazebo.urdf.xacro"/>
-    <xacro:include filename="$(find osr_gazebo)/urdf/insert_transmission.urdf.xacro"/>
+    <!-- Links and joint definitions -->
     <link name="base_footprint"/>
     <link name="base_link">
@@ -241,5 +240,4 @@
         </link>
         <joint name="front_wheel_joint_${prefix}" type="revolute">
-        <!-- revolute continuous -->
             <parent link="rocker_bogie_link_${prefix}_2"/>
             <origin rpy="0 0 0" xyz="0.170113 -0.000335 0.076721"/>
@@ -252,5 +250,4 @@
                 <origin rpy="${origin} 0 ${-dir*1.57}" xyz="0 0 0.0"/>
                 <geometry>
-                    <!-- <cylinder radius="0.03" length="0.04"/> -->
                     <mesh filename="file://$(find osr_gazebo)/simplified_meshes/wheel_middle_left.stl"/>
                 </geometry>
@@ -259,5 +256,4 @@
                 <origin rpy="${origin} 0 ${-dir*1.57}" xyz="0 0 0.0"/>
                 <geometry>
-                    <!-- <cylinder radius="0.03" length="0.04"/> -->
                     <mesh filename="file://$(find osr_gazebo)/simplified_meshes/wheel_middle_left.stl"/>
                 </geometry>
@@ -280,5 +276,4 @@
                 <origin rpy="0 0 ${-dir*1.57}" xyz="0 0 0.0"/>
                 <geometry>
-                    <!-- <cylinder radius="0.03" length="0.04"/> -->
                     <mesh filename="file://$(find osr_gazebo)/simplified_meshes/wheel_link_left_2.stl"/>
                 </geometry>
@@ -287,5 +282,4 @@
                 <origin rpy="0 0 ${-dir*1.57}" xyz="0 0 0.0"/>
                 <geometry>
-                    <!-- <cylinder radius="0.03" length="0.04"/> -->
                     <mesh filename="file://$(find osr_gazebo)/simplified_meshes/wheel_link_left_2.stl"/>
                 </geometry>
@@ -299,5 +293,4 @@
         </link>
         <joint name="rear_wheel_joint_${prefix}" type="revolute">
-        <!-- revolute continuous -->
             <parent link="rocker_bogie_link_${prefix}_1"/>
             <origin rpy="0 0 0" xyz="-0.311763 0 -0.030379"/>
@@ -314,6 +307,5 @@
                 <origin rpy="-1.57 0 ${origin}" xyz="0 0 0.0"/>
                 <geometry>
-                    <cylinder radius="0.082" length="0.04"/>
-                    <!-- <mesh filename="file://$(find osr_gazebo)/simplified_meshes/wheel.stl"/> -->
+                    <mesh filename="file://$(find osr_gazebo)/simplified_meshes/wheel.stl"/>
                 </geometry>
                 <surface>
@@ -329,6 +321,5 @@
                 <origin rpy="-1.57 0 ${origin}" xyz="0 0 0.0"/>
                 <geometry>
-                    <cylinder radius="0.082" length="0.04"/>
-                    <!-- <mesh filename="file://$(find osr_gazebo)/simplified_meshes/wheel.stl"/> -->
+                    <mesh filename="file://$(find osr_gazebo)/simplified_meshes/wheel.stl"/>
                 </geometry>
                 <material name="black"/>
@@ -351,6 +342,5 @@
                 <origin rpy="-1.57 0 ${origin}" xyz="0 0 0.0"/>
                 <geometry>
-                    <cylinder radius="0.082" length="0.04"/>
-                    <!-- <mesh filename="file://$(find osr_gazebo)/simplified_meshes/wheel.stl"/> -->
+                    <mesh filename="file://$(find osr_gazebo)/simplified_meshes/wheel.stl"/>
                 </geometry>
                 <surface>
@@ -366,6 +356,5 @@
                 <origin rpy="-1.57 0 ${origin}" xyz="0 0 0.0"/>
                 <geometry>
-                    <cylinder radius="0.082" length="0.04"/>
-                    <!-- <mesh filename="file://$(find osr_gazebo)/simplified_meshes/wheel.stl"/> -->
+                    <mesh filename="file://$(find osr_gazebo)/simplified_meshes/wheel.stl"/>
                 </geometry>
                 <material name="black"/>
@@ -388,6 +377,5 @@
                 <origin rpy="-1.57 0 ${origin}" xyz="0 0 0.0"/>
                 <geometry>
-                    <cylinder radius="0.082" length="0.04"/>
-                    <!-- <mesh filename="file://$(find osr_gazebo)/simplified_meshes/wheel.stl"/> -->
+                    <mesh filename="file://$(find osr_gazebo)/simplified_meshes/wheel.stl"/>
                 </geometry>
                 <surface>
@@ -403,6 +391,5 @@
                 <origin rpy="-1.57 0 ${origin}" xyz="0 0 0.0"/>
                 <geometry>
-                    <cylinder radius="0.082" length="0.04"/>
-                    <!-- <mesh filename="file://$(find osr_gazebo)/simplified_meshes/wheel.stl"/> -->
+                    <mesh filename="file://$(find osr_gazebo)/simplified_meshes/wheel.stl"/>
                 </geometry>
                 <material name="black"/>
@@ -424,10 +411,4 @@
     <xacro:wheel prefix="left" dir="1" origin="0" prefix_1="L"/>
     <xacro:wheel prefix="right" dir="-1" origin="3.14" prefix_1="R"/>
-    <joint name="imu_joint" type="fixed">
-            <parent link="base_link"/>
-            <child link="imu_link"/>
-            <origin xyz="0 0 0" rpy="0 0 0"/>
-        </joint>
-    <link name="imu_link"></link>
     <xacro:insert_velocity_transmission name="rear_wheel_joint_right"/>
     <xacro:insert_velocity_transmission name="rear_wheel_joint_left"/>
@@ -440,52 +421,5 @@
     <xacro:insert_position_transmission name="rear_wheel_joint_R"/>
     <xacro:insert_position_transmission name="rear_wheel_joint_L"/>
-    <joint name="laser_joint" type="fixed">
-        <parent link="base_link" />
-        <child link="laser_frame" />
-        <origin xyz="0.09 0 0.085" rpy="0 0 0" />
-    </joint>
-    <link name="laser_frame">
-        <visual>
-            <geometry>
-                <cylinder radius="0.03" length="0.04"/>
-            </geometry>
-            <material name="blue"/>
-        </visual>
-        <collision>
-            <geometry>
-                <cylinder radius="0.03" length="0.04"/>
-            </geometry>
-        </collision>
-    </link>
-    <gazebo reference="laser_frame">
-        <sensor name="laser" type="ray">
-            <pose>0 0 0 0 0 0</pose>
-            <visualize>false</visualize>
-            <update_rate>10</update_rate>
-            <ray>
-                <scan>
-                    <horizontal>
-                        <samples>720</samples>
-                        <resolution>1</resolution> <!--(max_angle-min_angle)/samples * resolution -->
-                        <min_angle>-3.14159</min_angle>
-                        <max_angle>3.14159</max_angle>
-                    </horizontal>
-                </scan>
-                <range>
-                    <min>0.3</min>
-                    <max>12.0</max>
-                    <resolution>0.01</resolution>
-                </range>
-                <noise>
-                    <type>gaussian</type>
-                    <mean>0.0</mean>
-                    <stddev>0.01</stddev>
-                </noise>
-            </ray>
-            <plugin name="laser_controller" filename="libgazebo_ros_ray_sensor.so">
-                <output_type>sensor_msgs/LaserScan</output_type>
-                <frame_name>laser_frame</frame_name>
-            </plugin>
-        </sensor>
-    </gazebo>
+    <!-- Add here IMU link and joint -->
+    <!-- Add here LiDAR link and joint -->
 </robot>
